File: hardware/sidewinder-usb/sidewinder-usb.kicad_pcb (KiCad board)
At the start: 2 copper layers, 40 x 55 mm, 22 parts, among them J1 USB_B_Micro, J2 DB15_Female, SW1 Reset, U1 ATmega32U4-AU, Y1 16MHz

Commit message: Final design for v0.2
Other:
- board text added: "Sidewinder USB Adapter v0.2"
Changed lines of the file:
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@@
   (general
     (thickness 1.6)
-    (drawings 4)
+    (drawings 5)
     (tracks 119)
     (zones 0)
@@
     (user_trace_width 1)
     (trace_clearance 0.2)
-    (zone_clearance 0.508)
+    (zone_clearance 0.1)
     (zone_45_only no)
     (trace_min 0.2)
@@
     (visible_elements FFFFFF7F)
     (pcbplotparams
-      (layerselection 0x010fc_ffffffff)
+      (layerselection 0x010f8_ffffffff)
       (usegerberextensions false)
       (usegerberattributes false)
@@
     (add_net VCC)
   )
+  (module sidewinder-usb:Auris_HC49USSMD (layer F.Cu)
+    (at 34 -20 90)
+    (fp_text reference Y1 (at 7 -2) (layer F.SilkS)
+      (effects (font (size 1 1) (thickness 0.15)))
+    )
+    (fp_text value 16MHz (at 0 -4 90) (layer F.Fab) hide
+      (effects (font (size 1 1) (thickness 0.15)))
+    )
+    (fp_line (start 5.7 -2.4) (end 5.7 2.4) (layer F.SilkS) (width 0.12))
+    (fp_line (start -5.7 -2.4) (end -5.7 2.4) (layer F.SilkS) (width 0.12))
+    (fp_line (start -5.7 2.4) (end 5.7 2.4) (layer F.SilkS) (width 0.12))
+    (fp_line (start -5.7 -2.4) (end 5.7 -2.4) (layer F.SilkS) (width 0.12))
+    (fp_line (start -6.5 -2.4) (end 6.5 -2.4) (layer F.Fab) (width 0.12))
+    (fp_line (start 6.5 -2.4) (end 6.5 2.4) (layer F.Fab) (width 0.12))
+    (fp_line (start 6.5 2.4) (end -6.5 2.4) (layer F.Fab) (width 0.12))
+    (fp_line (start -6.5 2.4) (end -6.5 -2.4) (layer F.Fab) (width 0.12))
+    (pad 2 smd rect (at 4.25 0 90) (size 4.5 2) (layers F.Cu F.Paste F.Mask)
+      (net 4 "Net-(C4-Pad1)"))
+    (pad 1 smd rect (at -4.25 0 90) (size 4.5 2) (layers F.Cu F.Paste F.Mask)
+      (net 3 "Net-(C3-Pad1)"))
+  )
   (module MountingHole:MountingHole_3.2mm_M3 (layer F.Cu)
     (at 35 -35)
@@
     )
     (pad 1 np_thru_hole circle (at 0 0) (size 3.2 3.2) (drill 3.2) (layers *.Cu *.Mask))
-  )
-  (module sidewinder-usb:Auris_HC49USSMD (layer F.Cu)
-    (at 34 -20 90)
-    (fp_text reference Y1 (at 0 4 90) (layer F.SilkS)
-      (effects (font (size 1 1) (thickness 0.15)))
-    )
-    (fp_text value 16MHz (at 0 -4 90) (layer F.Fab) hide
-      (effects (font (size 1 1) (thickness 0.15)))
-    )
-    (fp_line (start 5.7 -2.4) (end 5.7 2.4) (layer F.SilkS) (width 0.12))
-    (fp_line (start -5.7 -2.4) (end -5.7 2.4) (layer F.SilkS) (width 0.12))
-    (fp_line (start -5.7 2.4) (end 5.7 2.4) (layer F.SilkS) (width 0.12))
-    (fp_line (start -5.7 -2.4) (end 5.7 -2.4) (layer F.SilkS) (width 0.12))
-    (pad 2 smd rect (at 4.25 0 90) (size 4.5 2) (layers F.Cu F.Paste F.Mask)
-      (net 4 "Net-(C4-Pad1)"))
-    (pad 1 smd rect (at -4.25 0 90) (size 4.5 2) (layers F.Cu F.Paste F.Mask)
-      (net 3 "Net-(C3-Pad1)"))
   )
   (module Package_QFP:TQFP-44_10x10mm_P0.8mm (layer F.Cu)
@@
       (effects (font (size 1 1) (thickness 0.15)))
     )
-    (fp_text value Reset (at -5.76 0 180) (layer F.Fab)
+    (fp_text value Reset (at -5.76 0 180) (layer F.SilkS)
       (effects (font (size 1 1) (thickness 0.15)))
     )
@@
       (effects (font (size 1 1) (thickness 0.15)))
     )
-    (fp_text value 2.2k (at -2.5 0 180) (layer F.Fab)
+    (fp_text value 2.2k (at -2.5 0 180) (layer F.SilkS)
       (effects (font (size 1 1) (thickness 0.15)))
     )
@@
       (effects (font (size 1 1) (thickness 0.15)))
     )
-    (fp_text value 2.2k (at -2.5 0 180) (layer F.Fab)
+    (fp_text value 2.2k (at -2.5 0 180) (layer F.SilkS)
       (effects (font (size 1 1) (thickness 0.15)))
     )
@@
       (effects (font (size 1 1) (thickness 0.15)))
     )
-    (fp_text value 10k (at 0 1.65) (layer F.Fab)
+    (fp_text value 10k (at 0 1.65) (layer F.SilkS)
       (effects (font (size 1 1) (thickness 0.15)))
     )
@@
       (effects (font (size 1 1) (thickness 0.15)))
     )
-    (fp_text value 22R (at 2.5 1.5 180) (layer F.Fab)
+    (fp_text value 22R (at 2.5 1.5 180) (layer F.SilkS)
       (effects (font (size 1 1) (thickness 0.15)))
     )
@@
       (effects (font (size 1 1) (thickness 0.15)))
     )
-    (fp_text value 22R (at 2.5 -1.5 180) (layer F.Fab)
+    (fp_text value 22R (at 2.5 -1.5 180) (layer F.SilkS)
       (effects (font (size 1 1) (thickness 0.15)))
     )
@@
       (effects (font (size 1 1) (thickness 0.15)))
     )
-    (fp_text value 2.2n (at -2.5 0 180) (layer F.Fab)
+    (fp_text value 2.2n (at -2.5 0 180) (layer F.SilkS)
       (effects (font (size 1 1) (thickness 0.15)))
     )
@@
       (effects (font (size 1 1) (thickness 0.15)))
     )
-    (fp_text value 2.2n (at -2.5 0 180) (layer F.Fab)
+    (fp_text value 2.2n (at -2.5 0 180) (layer F.SilkS)
       (effects (font (size 1 1) (thickness 0.15)))
     )
@@
       (effects (font (size 1 1) (thickness 0.15)))
     )
-    (fp_text value 1u (at 0.7 -2.1 180) (layer F.Fab)
+    (fp_text value 1u (at 0.7 -2.1 180) (layer F.SilkS)
       (effects (font (size 1 1) (thickness 0.15)))
     )
@@
     (tags capacitor)
     (attr smd)
-    (fp_text reference C4 (at -2.8 -0.6) (layer F.SilkS)
-      (effects (font (size 1 1) (thickness 0.15)))
-    )
-    (fp_text value 22p (at -3.2 1) (layer F.Fab)
+    (fp_text reference C4 (at 1.5 1.6) (layer F.SilkS)
+      (effects (font (size 1 1) (thickness 0.15)))
+    )
+    (fp_text value 22p (at -2 1.6) (layer F.SilkS)
       (effects (font (size 1 1) (thickness 0.15)))
     )
@@
     (tags capacitor)
     (attr smd)
-    (fp_text reference C3 (at -2.8 0.5) (layer F.SilkS)
-      (effects (font (size 1 1) (thickness 0.15)))
-    )
-    (fp_text value 22p (at -3.2 -1) (layer F.Fab)
+    (fp_text reference C3 (at 1.5 -1.6) (layer F.SilkS)
+      (effects (font (size 1 1) (thickness 0.15)))
+    )
+    (fp_text value 22p (at -2 -1.6) (layer F.SilkS)
       (effects (font (size 1 1) (thickness 0.15)))
     )
@@
       (effects (font (size 1 1) (thickness 0.15)))
     )
-    (fp_text value 100nF (at -2.45 0.35 180) (layer F.Fab)
+    (fp_text value 100nF (at -2.45 0.35 180) (layer F.SilkS)
       (effects (font (size 1 1) (thickness 0.15)))
     )
@@
       (effects (font (size 1 1) (thickness 0.15)))
     )
-    (fp_text value 10uF (at 0.5 2.75 180) (layer F.Fab)
+    (fp_text value 10uF (at 0.5 2.75 180) (layer F.SilkS)
       (effects (font (size 1 1) (thickness 0.15)))
     )
@@
       (rotate (xyz 0 0 0))
     )
+  )
+  (gr_text "Sidewinder USB Adapter v0.2" (at 39 -20 90) (layer F.SilkS)
+    (effects (font (size 1 1) (thickness 0.1)))
   )
   (gr_line (start 40 -55) (end 40 0) (layer Edge.Cuts) (width 0.1))
@@
     (connect_pads (clearance 0.1))
     (min_thickness 0.1)
-    (fill yes (arc_segments 32) (thermal_gap 0.1) (thermal_bridge_width 0.2))
+    (fill yes (arc_segments 32) (thermal_gap 0.2) (thermal_bridge_width 0.5))
     (polygon
       (pts
